File: components/mini-pcb-3-to-5V-booster/mini-pcb-3-to-5V-booster.kicad_sch (KiCad schematic)
At the start: 9 parts, among them J1 INPUT, J2 OUTPUT 5V, U1 MT3608

Commit message: Latest test before production
Parts:
- C1, C2: LCSC C1644 -> C602037
Changed lines of the file:
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@@
       (effects (font (size 1.27 1.27)) hide)
     )
-    (property "LCSC" "C1644" (id 4) (at 100.33 91.44 0)
+    (property "LCSC" "C602037" (id 4) (at 100.33 91.44 0)
       (effects (font (size 1.27 1.27)) hide)
     )
@@
       (effects (font (size 1.27 1.27)) hide)
     )
-    (property "LCSC" "C1644" (id 4) (at 163.83 86.36 0)
+    (property "LCSC" "C602037" (id 4) (at 163.83 86.36 0)
       (effects (font (size 1.27 1.27)) hide)
     )
